Commit message: Completely fixed URDF

File: src/practice_bot_description/urdf/practice_bot.urdf.xacro (robot description, xacro)
@@ -3,4 +3,9 @@
     <xacro:property name="PI" value="3.14259"/>
     <link name="world"/>
+    <joint name="virtual_joint" type="fixed">
+        <parent link="world"/>
+        <child link="base_link"/>
+        <origin rpy="0 0 0" xyz="0 0 0"/>
+    </joint>
     <link name="base_link">
         <visual>
@@ -11,12 +16,9 @@
         </visual>
     </link>
-    <joint name="virtual_joint" type="fixed">
-        <parent link="world"/>
-        <child link="base_link"/>
-        <origin rpy="0 0 0" xyz="0 0 0"/>
-    </joint>
+    <!-- First Arm Joint: Defines the actual pivot coordinate frame in RViz -->
     <link name="robot_first_arm">
         <visual>
-            <origin rpy="-${PI} 0 0" xyz="-0.86 -0.55 0.39"/>
+            <!-- Set to zero so the mesh perfectly aligns with the joint frame above -->
+            <origin rpy="${PI} 0 0" xyz="-0.12 0.21 0.2"/>
             <geometry>
                 <mesh filename="package://practice_bot_description/meshes/robot_first_arm.STL" scale="0.007 0.007 0.007"/>
@@ -27,11 +29,12 @@
         <parent link="base_link"/>
         <child link="robot_first_arm"/>
-        <origin rpy="0 0 0" xyz="0.25 0 0"/>
+        <origin rpy="0 0 0" xyz="0 -0.05 0.7"/>
         <axis xyz="0 1 0"/>
         <limit effort="100" lower="-1.57" upper="1.57" velocity="1.0"/>
     </joint>
-    <link name="robot_second_arm">
+      <link name="robot_second_arm">
         <visual>
-            <origin rpy="0 0 0" xyz="1.0 0.5 0.5"/>
+            <!-- Set to zero to prevent the 'double-move' issue -->
+            <origin rpy="${PI} 0 0" xyz="-0.153 0.24 0.18"/>
             <geometry>
                 <mesh filename="package://practice_bot_description/meshes/robot_second_arm.STL" scale="0.007 0.007 0.007"/>
@@ -39,8 +42,9 @@
         </visual>
     </link>
+    <!-- Second Arm Joint: Defines the actual pivot coordinate frame in RViz -->
     <joint name="robot_second_arm_joint" type="revolute">
         <parent link="robot_first_arm"/>
         <child link="robot_second_arm"/>
-        <origin rpy="0 0 0" xyz="1.0 0.5 0.5"/>
+        <origin rpy="0 0 0" xyz="1.23 0.14 0"/>
         <axis xyz="0 1 0"/>
         <limit effort="100" lower="-1.57" upper="1.57" velocity="1.0"/>
